File: ExpressionInput.kicad_sch (KiCad schematic)
At the start: 8 parts

Commit message: Update
Parts:
- gave numbers to parts that had none: 2
- renumbered C101 to C301, R104 to R301, R104 to R302, R104 to R303
Changed lines of the file:
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@@
   (title_block
     (title "Expression Input")
-    (date "2023-06-03")
+    (date "2024-01-03")
     (rev "2")
     (company "Versio Duo")
@@
   (symbol (lib_id "Device:R_Small") (at 140.97 93.98 180) (unit 1)
     (in_bom yes) (on_board yes) (dnp no)
-    (property "Reference" "R104" (at 143.51 92.7101 0)
+    (property "Reference" "R301" (at 143.51 92.7101 0)
       (effects (font (size 1.27 1.27)) (justify right))
     )
@@
     (instances
       (project "express"
-        (path "/6c8448b4-b04d-47e1-934e-e40cbe27a7be"
-          (reference "R104") (unit 1)
-        )
         (path "/6c8448b4-b04d-47e1-934e-e40cbe27a7be/970e7b1b-3d39-40bf-a881-e4c7b552e176"
           (reference "R301") (unit 1)
@@
   (symbol (lib_id "Device:R_Small") (at 154.94 101.6 270) (unit 1)
     (in_bom yes) (on_board yes) (dnp no)
-    (property "Reference" "R104" (at 157.4801 104.14 90)
+    (property "Reference" "R302" (at 157.4801 104.14 90)
       (effects (font (size 1.27 1.27)) (justify right))
     )
@@
     (instances
       (project "express"
-        (path "/6c8448b4-b04d-47e1-934e-e40cbe27a7be"
-          (reference "R104") (unit 1)
-        )
         (path "/6c8448b4-b04d-47e1-934e-e40cbe27a7be/970e7b1b-3d39-40bf-a881-e4c7b552e176"
           (reference "R302") (unit 1)
@@
   (symbol (lib_id "V2_Connector_Audio:SJ2-25504B-SMT-TR") (at 109.22 100.33 0) (mirror y) (unit 1)
     (in_bom yes) (on_board yes) (dnp no)
-    (property "Reference" "J?" (at 101.6 85.725 0)
+    (property "Reference" "J301" (at 101.6 85.725 0)
       (effects (font (size 1.27 1.27)) (justify left))
     )
@@
     (instances
       (project "express"
-        (path "/6c8448b4-b04d-47e1-934e-e40cbe27a7be"
-          (reference "J?") (unit 1)
-        )
         (path "/6c8448b4-b04d-47e1-934e-e40cbe27a7be/970e7b1b-3d39-40bf-a881-e4c7b552e176"
           (reference "J301") (unit 1)
@@
   (symbol (lib_id "Device:C_Small") (at 198.12 104.14 0) (unit 1)
     (in_bom yes) (on_board yes) (dnp no)
-    (property "Reference" "C101" (at 207.01 104.14 0)
+    (property "Reference" "C301" (at 207.01 104.14 0)
       (effects (font (size 1.27 1.27)) (justify right))
     )
@@
     (instances
       (project "express"
-        (path "/6c8448b4-b04d-47e1-934e-e40cbe27a7be"
-          (reference "C101") (unit 1)
-        )
         (path "/6c8448b4-b04d-47e1-934e-e40cbe27a7be/970e7b1b-3d39-40bf-a881-e4c7b552e176"
           (reference "C301") (unit 1)
@@
   (symbol (lib_id "V2_LED:WS2812") (at 156.21 138.43 0) (unit 1)
     (in_bom yes) (on_board yes) (dnp no)
-    (property "Reference" "D?" (at 153.67 128.27 0)
+    (property "Reference" "D301" (at 153.67 128.27 0)
       (effects (font (size 1.27 1.27)))
     )
@@
     (instances
       (project "express"
-        (path "/6c8448b4-b04d-47e1-934e-e40cbe27a7be"
-          (reference "D?") (unit 1)
-        )
         (path "/6c8448b4-b04d-47e1-934e-e40cbe27a7be/970e7b1b-3d39-40bf-a881-e4c7b552e176"
           (reference "D301") (unit 1)
@@
   (symbol (lib_id "Device:R_Small") (at 140.97 104.14 0) (unit 1)
     (in_bom yes) (on_board yes) (dnp no)
-    (property "Reference" "R104" (at 148.59 104.1399 0)
+    (property "Reference" "R303" (at 148.59 104.1399 0)
       (effects (font (size 1.27 1.27)) (justify right))
     )
@@
     (instances
       (project "express"
-        (path "/6c8448b4-b04d-47e1-934e-e40cbe27a7be"
-          (reference "R104") (unit 1)
-        )
         (path "/6c8448b4-b04d-47e1-934e-e40cbe27a7be/970e7b1b-3d39-40bf-a881-e4c7b552e176"
           (reference "R303") (unit 1)
