File: express.kicad_pcb (KiCad board)
At the start: 4 copper layers, 180 x 35 mm, 180 parts, among them J1001 SJ2-25504B-SMT-TR, J101 Cortex_Debug, J102 JAE_DX07S016JA3, J1101 SJ2-25504B-SMT-TR, J1201 SJ2-25504B-SMT-TR, J1301 SJ2-25504B-SMT-TR, J1401 SJ2-25504B-SMT-TR, J1501 SJ2-25504B-SMT-TR, J1601 SJ2-25504B-SMT-TR, J1701 SJ2-25504B-SMT-TR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

Commit message: Replace MIDI In with MIDI Out
Parts:
- removed C201, C202: 0u1, Capacitor_SMD:C_0603_1608Metric
- added R202: 220R, Resistor_SMD:R_0603_1608Metric, F.Cu at (66.2, 99.5)
- added TVS201: CG0603MLC-05LE, Diode_SMD:D_0603_1608Metric, F.Cu at (66.2, 101.2)
- U201: value TLP2361 -> 74AHC1G125; footprint Package_SO:SO-6_4.4x3.6mm_P1.27mm -> Package_TO_SOT_SMD:SOT-23-5
- moved D201 18.4 mm to (66.2, 98.0)
- moved U201 14.7 mm to (70.0, 100.8), turned to 180 degrees
- moved R201 12.2 mm to (69.2, 98.0), turned to 0 degrees
Connections:
- D201 pad 1: Net-(D201-K) -> /MIDI Out/Ring
- D201 pad 2: /MIDI In/Tip -> Net-(D201-A)
- J201 pad 1: Net-(J201-S) -> GND
- J201 pad 3: /MIDI In/Ring -> /MIDI Out/Ring
- J201 pad 5: /MIDI In/Tip -> /MIDI Out/Tip
- R201 pad 1: /MIDI In/Ring -> Net-(TVS201-A)
- R201 pad 2: Net-(D201-K) -> /MIDI Out/Tip
- U103 pad 13: /Button -> /MIDI-Out
- U103 pad 14: /MIDI-In -> unconnected-(U103-PA05-Pad14)
- U103 pad 30: unconnected-(U103-PA13-Pad30) -> /Button
- U201 pad 1: Net-(D201-K) -> /MIDI-Out
- U201 pad 2: unconnected-(U201-NC-Pad2) -> GND
- U201 pad 3: /MIDI In/Tip -> GND
- U201 pad 4: GND -> Net-(TVS201-A)
- U201 pad 5: /MIDI-In -> +5V
Routing:
- net /MIDI-Out: track 0.00 -> 31.2 mm
- net /MIDI In/Tip: track 20.8 -> 0.00 mm
- net /MIDI In/Ring: track 16.5 -> 0.00 mm
- net /MIDI-In: track 14.3 -> 0.00 mm
- net /Button: track 67.0 -> 58.5 mm
- net Net-(D201-K): track 5.28 -> 0.00 mm
- net Net-(TVS201-A): track 0.00 -> 4.38 mm
- net +3V3: track 31.5 -> 28.3 mm, vias 27 -> 26
- net /MIDI Out/Ring: track 0.00 -> 2.90 mm
- net /MIDI Out/Tip: track 0.00 -> 2.36 mm
- net Net-(J201-S): track 2.26 -> 0.00 mm
- net Net-(D201-A): track 0.00 -> 1.55 mm
- net +5V: track 20.2 -> 21.5 mm, vias 27 -> 29

Commit message: Refresh
Parts:
- INFO101: value Order_Number -> ORDER-NUMBER
Changed lines of the file:
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@@
   (paper "A4")
   (title_block
-    (date "2023-06-03")
+    (date "2023-07-01")
     (rev "3")
   )
@@
     (fp_line (start 4.5 4.5) (end -4.5 4.5)
       (stroke (width 0.1) (type solid)) (layer "F.Fab"))
-    (pad "" smd roundrect (at -1.4 -1.4 270) (size 1.263087 1.263087) (layers "F.Paste") (roundrect_rratio 0.197928))
-    (pad "" smd roundrect (at -1.4 0 270) (size 1.263087 1.263087) (layers "F.Paste") (roundrect_rratio 0.197928))
-    (pad "" smd roundrect (at -1.4 1.4 270) (size 1.263087 1.263087) (layers "F.Paste") (roundrect_rratio 0.197928))
-    (pad "" smd roundrect (at 0 -1.4 270) (size 1.263087 1.263087) (layers "F.Paste") (roundrect_rratio 0.197928))
-    (pad "" smd roundrect (at 0 0 270) (size 1.263087 1.263087) (layers "F.Paste") (roundrect_rratio 0.197928))
-    (pad "" smd roundrect (at 0 1.4 270) (size 1.263087 1.263087) (layers "F.Paste") (roundrect_rratio 0.197928))
-    (pad "" smd roundrect (at 1.4 -1.4 270) (size 1.263087 1.263087) (layers "F.Paste") (roundrect_rratio 0.197928))
-    (pad "" smd roundrect (at 1.4 0 270) (size 1.263087 1.263087) (layers "F.Paste") (roundrect_rratio 0.197928))
-    (pad "" smd roundrect (at 1.4 1.4 270) (size 1.263087 1.263087) (layers "F.Paste") (roundrect_rratio 0.197928))
+    (pad "" smd roundrect (at -1.4 -1.4 270) (size 1.15 1.15) (layers "F.Paste") (roundrect_rratio 0.1))
+    (pad "" smd roundrect (at -1.4 0 270) (size 1.15 1.15) (layers "F.Paste") (roundrect_rratio 0.1))
+    (pad "" smd roundrect (at -1.4 1.4 270) (size 1.15 1.15) (layers "F.Paste") (roundrect_rratio 0.1))
+    (pad "" smd roundrect (at 0 -1.4 270) (size 1.15 1.15) (layers "F.Paste") (roundrect_rratio 0.1))
+    (pad "" smd roundrect (at 0 0 270) (size 1.15 1.15) (layers "F.Paste") (roundrect_rratio 0.1))
+    (pad "" smd roundrect (at 0 1.4 270) (size 1.15 1.15) (layers "F.Paste") (roundrect_rratio 0.1))
+    (pad "" smd roundrect (at 1.4 -1.4 270) (size 1.15 1.15) (layers "F.Paste") (roundrect_rratio 0.1))
+    (pad "" smd roundrect (at 1.4 0 270) (size 1.15 1.15) (layers "F.Paste") (roundrect_rratio 0.1))
+    (pad "" smd roundrect (at 1.4 1.4 270) (size 1.15 1.15) (layers "F.Paste") (roundrect_rratio 0.1))
     (pad "1" smd roundrect (at -4.4125 -3.75 270) (size 0.875 0.2) (layers "F.Cu" "F.Paste" "F.Mask") (roundrect_rratio 0.25)
       (net 29 "/XIN32") (pinfunction "PA00") (pintype "bidirectional"))
@@
         (effects (font (size 1 1) (thickness 0.15)))
     )
-    (fp_text value "Order_Number" (at 0 2.27 unlocked) (layer "F.Fab") hide
+    (fp_text value "ORDER-NUMBER" (at 0 2.27 unlocked) (layer "F.Fab") hide
         (effects (font (size 1 1) (thickness 0.15)))
     )
@@
     (fp_line (start 1.5 1.5) (end -1.5 1.5)
       (stroke (width 0.1) (type solid)) (layer "F.Fab"))
-    (pad "" smd rect (at -0.45 -0.625 270) (size 0.6 1) (layers "F.Paste"))
-    (pad "" smd rect (at -0.45 0.625 270) (size 0.6 1) (layers "F.Paste"))
-    (pad "" smd rect (at 0.45 -0.625 270) (size 0.6 1) (layers "F.Paste"))
-    (pad "" smd rect (at 0.45 0.625 270) (size 0.6 1) (layers "F.Paste"))
+    (pad "" smd roundrect (at -0.45 -0.625 270) (size 0.6 1) (layers "F.Paste") (roundrect_rratio 0.1))
+    (pad "" smd roundrect (at -0.45 0.625 270) (size 0.6 1) (layers "F.Paste") (roundrect_rratio 0.1))
+    (pad "" smd roundrect (at 0.45 -0.625 270) (size 0.6 1) (layers "F.Paste") (roundrect_rratio 0.1))
+    (pad "" smd roundrect (at 0.45 0.625 270) (size 0.6 1) (layers "F.Paste") (roundrect_rratio 0.1))
     (pad "1" smd rect (at -1.4 -0.975 270) (size 0.6 0.31) (layers "F.Cu" "F.Paste" "F.Mask")
       (net 3 "+3V3") (pinfunction "OUT") (pintype "power_out"))
@@
       )
     )
-    (group "" (id 6aa83fe3-45eb-46aa-a986-6b9d53808faa)
+    (group "" (id 0cda7142-3a28-44c2-8222-5e22d7ffb10c)
       (members
-        02ab5ce3-a4ec-4889-880c-f28dfc686826
-        0aa981ac-dfa1-437c-baeb-623f50b50e09
-        390c389d-3209-466b-b47b-091b3372794d
-        47946ee2-a99a-42f9-9af4-c98efdbc1b75
-        4a331480-e968-440b-8e1a-f0e463ec292f
-        841a9b72-3288-4262-ac23-45a0faced35a
-        c877bb3b-0a16-4d3b-bfe7-cba9ec2d44c0
-        df1c22ff-1c07-4de3-9119-c6de912e036e
+        26451119-93a7-4a98-9776-ec5c6d8494d9
+        38e28a19-9ac8-4022-a8f3-c1724ce761dd
+        59a73271-5af4-4529-8df5-80dd4cca3ede
+        81fd9f0a-c2b5-4718-ae35-98a456b55d47
+        96612a54-3d21-4e7f-ab6d-fd66191c423b
+        97f661b1-1d7a-4d38-b618-f6f2b7e61e9a
+        9974fe82-d436-4e30-9969-277f3e2c874f
+        9f53dbb4-93fc-49b4-a43f-ad57aa66c827
       )
     )
-    (group "" (id 67cae43f-077d-4752-9cba-cedb39780545)
+    (group "" (id 0f2f4c35-41e2-434e-8e75-c55b8373f0d2)
       (members
-        14509c0e-2e51-40f4-8646-55b392a6f5b4
-        3f09ba6e-6ff3-4818-a096-5d23135ed52b
-        41bbe9d4-a1c1-411d-b9ad-05030f494abd
-        5ecd19d6-1df3-440f-a488-ae23c2cdade0
-        6e4e37b4-3ec7-4825-a680-2e7ae46b368b
-        88919d52-1eaf-4f98-a804-e7f01e9ce1e5
-        dc62afbd-cef0-46d4-90a7-17bb1c3c7f40
-        f818fe37-1aec-482b-8cde-4ca4cb0e9adb
+        56ec08ae-dc52-4801-ae22-4ff843885560
+        62641cdb-b6b7-4edc-825a-48083fc4499f
+        819f1f41-9d43-4d91-8760-becb7de0d24e
+        8b4876eb-6b91-4542-9326-da7dc9d55096
+        aa0b137b-8bc7-4102-8d95-cd4c34fd83f5
+        afc1ecff-3f01-4661-9114-81295c35868e
+        afcc6c69-d10e-4676-9a8d-3bd2dc12b171
+        f675512a-8f87-41b9-b5a5-ba989581218c
       )
     )
