File: express.kicad_sch (KiCad schematic)
At the start: 46 parts, among them J101 Cortex_Debug, J102 JAE_DX07S016JA3, SW101 SW_Push, SW102 SW_Push, U101 TPS78433QWDRBRQ1, U103 ATSAMD51J, Y102 32k768

Commit message: Replace MIDI In with MIDI Out
Connections:
- net Button: now also U103.30 (PA13); no longer U103.13 (PA04)
- net MIDI-In: no longer names the net of U103.14 (PA05)
- new net MIDI-Out: U103.13 (PA04)
Other:
- sheet MIDI In renamed MIDI Out
- sheet MIDI Out: file MIDIIn.kicad_sch -> MIDIOut.kicad_sch
- moved on the sheet: TVS101
Changed lines of the file:
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@@
   )
   (no_connect (at 53.34 82.55))
-  (no_connect (at 53.34 72.39))
   (no_connect (at 53.34 80.01))
+  (no_connect (at 53.34 52.07))
   (no_connect (at 86.36 82.55))
   (no_connect (at 53.34 90.17))
@@
     (stroke (width 0) (type default))
   )
+  (wire (pts (xy 34.29 49.53) (xy 53.34 49.53))
+    (stroke (width 0) (type default))
+  )
   (wire (pts (xy 72.39 20.32) (xy 72.39 31.75))
     (stroke (width 0) (type default))
@@
     (stroke (width 0) (type default))
   )
-  (wire (pts (xy 34.29 49.53) (xy 53.34 49.53))
-    (stroke (width 0) (type default))
-  )
   (wire (pts (xy 69.85 125.73) (xy 72.39 125.73))
     (stroke (width 0) (type default))
@@
   )
   (wire (pts (xy 137.16 55.88) (xy 134.62 55.88))
-    (stroke (width 0) (type default))
-  )
-  (wire (pts (xy 34.29 52.07) (xy 53.34 52.07))
     (stroke (width 0) (type default))
   )
@@
     (stroke (width 0) (type default))
   )
-  (wire (pts (xy 142.24 142.24) (xy 153.67 142.24))
+  (wire (pts (xy 123.19 142.24) (xy 111.76 142.24))
     (stroke (width 0) (type default))
   )
@@
   )
   (wire (pts (xy 67.31 125.73) (xy 69.85 125.73))
+    (stroke (width 0) (type default))
+  )
+  (wire (pts (xy 34.29 72.39) (xy 53.34 72.39))
     (stroke (width 0) (type default))
   )
@@
     (effects (font (size 1.27 1.27)) (justify left bottom))
   )
+  (label "Button" (at 34.29 72.39 0) (fields_autoplaced)
+    (effects (font (size 1.27 1.27)) (justify left bottom))
+  )
   (label "LED-onboard" (at 34.29 105.41 0) (fields_autoplaced)
     (effects (font (size 1.27 1.27)) (justify left bottom))
@@
     (effects (font (size 1.27 1.27)) (justify right bottom))
   )
-  (label "MIDI-In" (at 153.67 142.24 180) (fields_autoplaced)
-    (effects (font (size 1.27 1.27)) (justify right bottom))
+  (label "MIDI-Out" (at 111.76 142.24 0) (fields_autoplaced)
+    (effects (font (size 1.27 1.27)) (justify left bottom))
   )
   (label "Analog-2" (at 90.17 152.4 180) (fields_autoplaced)
@@
     (effects (font (size 1.27 1.27)) (justify left bottom))
   )
+  (label "MIDI-Out" (at 34.29 49.53 0) (fields_autoplaced)
+    (effects (font (size 1.27 1.27)) (justify left bottom))
+  )
   (label "Analog-3" (at 121.92 152.4 180) (fields_autoplaced)
     (effects (font (size 1.27 1.27)) (justify right bottom))
-  )
-  (label "Button" (at 34.29 49.53 0) (fields_autoplaced)
-    (effects (font (size 1.27 1.27)) (justify left bottom))
   )
   (label "LED-13" (at 16.51 193.04 0) (fields_autoplaced)
@@
   )
   (label "SWDIO" (at 34.29 110.49 0) (fields_autoplaced)
-    (effects (font (size 1.27 1.27)) (justify left bottom))
-  )
-  (label "MIDI-In" (at 34.29 52.07 0) (fields_autoplaced)
     (effects (font (size 1.27 1.27)) (justify left bottom))
   )
@@
     )
   )
-  (symbol (lib_id "V2_Diode:CG0603MLC-3.3LE") (at 100.33 142.24 0) (unit 1)
-    (in_bom yes) (on_board yes) (dnp no) (fields_autoplaced)
-    (property "Reference" "TVS101" (at 100.33 135.89 0)
-      (effects (font (size 1.27 1.27)))
-    )
-    (property "Value" "CG0603MLC-3.3LE" (at 100.33 138.43 0)
-      (effects (font (size 1.27 1.27)))
-    )
-    (property "Footprint" "Diode_SMD:D_0603_1608Metric" (at 100.33 147.955 0)
+  (symbol (lib_id "V2_Diode:CG0603MLC-3.3LE") (at 68.58 142.24 0) (unit 1)
+    (in_bom yes) (on_board yes) (dnp no) (fields_autoplaced)
+    (property "Reference" "TVS101" (at 68.58 135.89 0)
+      (effects (font (size 1.27 1.27)))
+    )
+    (property "Value" "CG0603MLC-3.3LE" (at 68.58 138.43 0)
+      (effects (font (size 1.27 1.27)))
+    )
+    (property "Footprint" "Diode_SMD:D_0603_1608Metric" (at 68.58 147.955 0)
       (effects (font (size 0 0)) hide)
     )
-    (property "Datasheet" "" (at 100.33 142.24 0)
+    (property "Datasheet" "" (at 68.58 142.24 0)
       (effects (font (size 1.27 1.27)) hide)
     )
@@
     )
   )
-  (symbol (lib_id "power:+3V3") (at 96.52 142.24 90) (unit 1)
-    (in_bom yes) (on_board yes) (dnp no) (fields_autoplaced)
-    (property "Reference" "#PWR0106" (at 100.33 142.24 0)
-      (effects (font (size 1.27 1.27)) hide)
-    )
-    (property "Value" "+3V3" (at 92.71 142.2399 90)
-      (effects (font (size 1.27 1.27)) (justify left))
-    )
-    (property "Footprint" "" (at 96.52 142.24 0)
-      (effects (font (size 1.27 1.27)) hide)
-    )
-    (property "Datasheet" "" (at 96.52 142.24 0)
+  (symbol (lib_id "power:+3V3") (at 64.77 142.24 90) (unit 1)
+    (in_bom yes) (on_board yes) (dnp no) (fields_autoplaced)
+    (property "Reference" "#PWR0106" (at 68.58 142.24 0)
+      (effects (font (size 1.27 1.27)) hide)
+    )
+    (property "Value" "+3V3" (at 60.96 142.2399 90)
+      (effects (font (size 1.27 1.27)) (justify left))
+    )
+    (property "Footprint" "" (at 64.77 142.24 0)
+      (effects (font (size 1.27 1.27)) hide)
+    )
+    (property "Datasheet" "" (at 64.77 142.24 0)
       (effects (font (size 1.27 1.27)) hide)
     )
@@
     )
   )
-  (symbol (lib_id "power:GND") (at 104.14 142.24 90) (unit 1)
-    (in_bom yes) (on_board yes) (dnp no) (fields_autoplaced)
-    (property "Reference" "#PWR0105" (at 110.49 142.24 0)
-      (effects (font (size 1.27 1.27)) hide)
-    )
-    (property "Value" "GND" (at 107.95 142.2399 90)
-      (effects (font (size 1.27 1.27)) (justify right))
-    )
-    (property "Footprint" "" (at 104.14 142.24 0)
-      (effects (font (size 1.27 1.27)) hide)
-    )
-    (property "Datasheet" "" (at 104.14 142.24 0)
+  (symbol (lib_id "power:GND") (at 72.39 142.24 90) (unit 1)
+    (in_bom yes) (on_board yes) (dnp no) (fields_autoplaced)
+    (property "Reference" "#PWR0105" (at 78.74 142.24 0)
+      (effects (font (size 1.27 1.27)) hide)
+    )
+    (property "Value" "GND" (at 76.2 142.2399 90)
+      (effects (font (size 1.27 1.27)) (justify right))
+    )
+    (property "Footprint" "" (at 72.39 142.24 0)
+      (effects (font (size 1.27 1.27)) hide)
+    )
+    (property "Datasheet" "" (at 72.39 142.24 0)
       (effects (font (size 1.27 1.27)) hide)
     )
@@
     (stroke (width 0.1524) (type solid))
     (fill (color 0 0 0 0.0000))
-    (property "Sheetname" "MIDI In" (at 123.19 138.9884 0)
+    (property "Sheetname" "MIDI Out" (at 123.19 138.9884 0)
       (effects (font (size 1.27 1.27)) (justify left bottom))
     )
-    (property "Sheetfile" "MIDIIn.kicad_sch" (at 123.19 145.3646 0)
+    (property "Sheetfile" "MIDIOut.kicad_sch" (at 123.19 145.3646 0)
       (effects (font (size 1.27 1.27)) (justify left top) hide)
     )
-    (pin "MIDI-Data" output (at 142.24 142.24 0)
-      (effects (font (size 1.27 1.27)) (justify right))
-    )
-    (instances
+    (pin "MIDI-Data" output (at 123.19 142.24 180)
+      (effects (font (size 1.27 1.27)) (justify left))
+    )
+    (instances

Commit message: Update
Other:
- moved on the sheet: ICON101
Changed lines of the file:
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@@
   (title_block
     (title "V2 express")
-    (date "2023-06-03")
+    (date "2024-01-03")
     (rev "3")
     (company "Versio Duo")
