File: LinkPlug.kicad_sch (KiCad schematic)
At the start: 6 parts, among them J1801 2x05_Horizontal, U1801 SN65MLVD203B

Commit message: Update tranceiver
Parts:
- removed R1801, R1803: 10k, Resistor_SMD:R_0603_1608Metric, symbol Device:R_Small
- U1801: value SN65MLVD203B -> THVD24x2; footprint V2_Package_DFN_QFN:WQFN-16-1EP_4x4mm_P0.65mm_EP2.7x2.7mm_ThermalVias -> V2_Package_SON:VSON-10-4-1EP_3x3mm_P0.5mm_EP1.65x2.4mm_ThermalVias; symbol V2_Interface_LVDS:SN65MLVD203B -> V2_Interface_RS485:THVD24x2
- renumbered R1802 to R1801
Connections:
- net +3V3: now also U1801.10 (VCC); no longer U1801.13 (VCC), U1801.14 (VCC)
- net GND: now also U1801.11 (GND); no longer U1801.17 (GND), U1801.6 (GND)
- net RX-A: now also U1801.9 (A); no longer U1801.12 (A)
- net RX-B: now also U1801.8 (B); no longer U1801.11 (B)
- net TX-Y: now also U1801.6 (Y); no longer U1801.9 (Y)
- net TX-Z: now also U1801.7 (Z); no longer U1801.10 (Z)

Commit message: Link termination
Parts:
- R1801: value 120R -> 100R
Changed lines of the file:
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@@
 			)
 		)
-		(property "Value" "120R"
+		(property "Value" "100R"
 			(at 153.67 109.22 0)
 			(effects
@@
 		(at 148.59 143.51 0)
 		(unit 1)
-		(exclude_from_sim no)
+		(exclude_from_sim yes)
 		(in_bom yes)
 		(on_board yes)
@@
 			(at 148.59 143.51 0)
 			(effects
-				(font
-					(size 1.27 1.27)
-				)
-				(hide yes)
-			)
-		)
-		(property "Sim.Enable" "0"
-			(at 148.59 143.51 0)
-			(effects
