File: express-cover/express-cover.kicad_pcb (KiCad board)
At the start: 2 copper layers, 180 x 35 mm, 26 parts

Commit message: Update
Parts:
- H101, H102, H103, H104, H105: value MountingHole_2mm_Pad_5.2mm -> Mounting_Hole; footprint V2_Mechanical:Mounting_Hole_2mm_Pad_5.2mm -> V2_Mechanical:MountingHole_2mm_Pad_5.2mm
- H107, H108, H109, H110, H111, H112, H113, H114, H115, H116, H117, H118, H119, H120, H121, H122: value MountingHole_2mm_Pad_2.4mm -> Mounting_Hole
- INFO101: value Order_Number -> ORDER-NUMBER
