File: express-cover/express-cover.kicad_pcb (KiCad board)
At the start: 2 copper layers, 180 x 35 mm, 26 parts

Commit message: Update tranceiver
Parts:
- H101: value Mounting_Hole -> MountingHole_2mm_Pad_5.2mm
- H102: renamed from H107; value Mounting_Hole -> MountingHole_2mm_Pad_2.4mm
- H103: renamed from H115; value Mounting_Hole -> MountingHole_2mm_Pad_2.4mm
- H104: renamed from H102; value Mounting_Hole -> MountingHole_2mm_Pad_5.2mm
- H105: renamed from H108; value Mounting_Hole -> MountingHole_2mm_Pad_2.4mm
- H106: renamed from H116; value Mounting_Hole -> MountingHole_2mm_Pad_2.4mm
- H107: renamed from H103; value Mounting_Hole -> MountingHole_2mm_Pad_5.2mm
- H108: renamed from H109; value Mounting_Hole -> MountingHole_2mm_Pad_2.4mm
- H109: renamed from H117; value Mounting_Hole -> MountingHole_2mm_Pad_2.4mm
- H110: renamed from H104; value Mounting_Hole -> MountingHole_2mm_Pad_5.2mm
- H111: renamed from H110; value Mounting_Hole -> MountingHole_2mm_Pad_2.4mm
- H112: renamed from H118; value Mounting_Hole -> MountingHole_2mm_Pad_2.4mm
- H113: renamed from H105; value Mounting_Hole -> MountingHole_2mm_Pad_5.2mm
- H114: renamed from H111; value Mounting_Hole -> MountingHole_2mm_Pad_2.4mm
- H115: renamed from H119; value Mounting_Hole -> MountingHole_2mm_Pad_2.4mm
- H116: renamed from H112; value Mounting_Hole -> MountingHole_2mm_Pad_2.4mm
- H117: renamed from H120; value Mounting_Hole -> MountingHole_2mm_Pad_2.4mm
- H118: renamed from H113; value Mounting_Hole -> MountingHole_2mm_Pad_2.4mm
- H119: renamed from H121; value Mounting_Hole -> MountingHole_2mm_Pad_2.4mm
- H120: renamed from H114; value Mounting_Hole -> MountingHole_2mm_Pad_2.4mm
- H121: renamed from H122; value Mounting_Hole -> MountingHole_2mm_Pad_2.4mm
- INFO101: value ORDER-NUMBER -> Order_Number
- moved H101 1.00 mm to (282.0, 85.0)
- moved H104 1.00 mm to (282.0, 110.0)
- moved H110 1.00 mm to (132.0, 85.0)
- moved H113 1.00 mm to (132.0, 110.0)
- moved ICON101 0.50 mm to (123.8, 110.0)
- moved ICON102 0.50 mm to (290.8, 110.0)
- renumbered H106 to H122, ICON102 to ICON101, ICON101 to ICON102
