File: express-cover/express-cover.kicad_sch (KiCad schematic)
At the start: 26 parts

Commit message: Update
Parts:
- H101, H102, H103, H104, H105: footprint V2_Mechanical:Mounting_Hole_2mm_Pad_5.2mm -> V2_Mechanical:MountingHole_2mm_Pad_5.2mm
Other:
- moved on the sheet: ICON102

Commit message: Use the correct TRS pins
Parts:
- H101, H102, H103, H104, H105, H106, H107, H108, H109, H110, H111, H112, H113, H114, H115, H116, H117, H118, H119, H120, H121, H122: now left out of the parts list
Changed lines of the file:
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@@
 		(unit 1)
 		(exclude_from_sim no)
-		(in_bom yes)
+		(in_bom no)
 		(on_board yes)
 		(dnp no)
@@
 		(unit 1)
 		(exclude_from_sim no)
-		(in_bom yes)
+		(in_bom no)
 		(on_board yes)
 		(dnp no)
@@
 		(unit 1)
 		(exclude_from_sim no)
-		(in_bom yes)
+		(in_bom no)
 		(on_board yes)
 		(dnp no)
@@
 		(unit 1)
 		(exclude_from_sim no)
-		(in_bom yes)
+		(in_bom no)
 		(on_board yes)
 		(dnp no)
@@
 		(unit 1)
 		(exclude_from_sim no)
-		(in_bom yes)
+		(in_bom no)
 		(on_board yes)
 		(dnp no)
@@
 		(unit 1)
 		(exclude_from_sim no)
-		(in_bom yes)
+		(in_bom no)
 		(on_board yes)
 		(dnp no)
@@
 		(unit 1)
 		(exclude_from_sim no)
-		(in_bom yes)
+		(in_bom no)
 		(on_board yes)
 		(dnp no)
@@
 		(unit 1)
 		(exclude_from_sim no)
-		(in_bom yes)
+		(in_bom no)
 		(on_board yes)
 		(dnp no)
@@
 		(unit 1)
 		(exclude_from_sim no)
-		(in_bom yes)
+		(in_bom no)
 		(on_board yes)
 		(dnp no)
@@
 		(unit 1)
 		(exclude_from_sim no)
-		(in_bom yes)
+		(in_bom no)
 		(on_board yes)
 		(dnp no)
@@
 		(unit 1)
 		(exclude_from_sim no)
-		(in_bom yes)
+		(in_bom no)
 		(on_board yes)
 		(dnp no)
@@
 		(unit 1)
 		(exclude_from_sim no)
-		(in_bom yes)
+		(in_bom no)
 		(on_board yes)
 		(dnp no)
@@
 		(unit 1)
 		(exclude_from_sim no)
-		(in_bom yes)
+		(in_bom no)
 		(on_board yes)
 		(dnp no)
@@
 		(unit 1)
 		(exclude_from_sim no)
-		(in_bom yes)
+		(in_bom no)
 		(on_board yes)
 		(dnp no)
@@
 		(unit 1)
 		(exclude_from_sim no)
-		(in_bom yes)
+		(in_bom no)
 		(on_board yes)
 		(dnp no)
@@
 		(unit 1)
 		(exclude_from_sim no)
-		(in_bom yes)
+		(in_bom no)
 		(on_board yes)
 		(dnp no)
@@
 		(unit 1)
 		(exclude_from_sim no)
-		(in_bom yes)
+		(in_bom no)
 		(on_board yes)
 		(dnp no)
@@
 		(unit 1)
 		(exclude_from_sim no)
-		(in_bom yes)
+		(in_bom no)
 		(on_board yes)
 		(dnp no)
@@
 		(unit 1)
 		(exclude_from_sim no)
-		(in_bom yes)
+		(in_bom no)
 		(on_board yes)
 		(dnp no)
@@
 		(unit 1)
 		(exclude_from_sim no)
-		(in_bom yes)
+		(in_bom no)
 		(on_board yes)
 		(dnp no)
@@
 		(unit 1)
 		(exclude_from_sim no)
-		(in_bom yes)
+		(in_bom no)
 		(on_board yes)
 		(dnp no)
@@
 		(unit 1)
 		(exclude_from_sim no)
-		(in_bom yes)
-		(on_board yes)
-		(dnp no)
+		(in_bom no)
+		(on_board yes)
+		(dnp no)

Commit message: Update tranceiver
Parts:
- renumbered H107 to H102, H115 to H103, H102 to H104, H108 to H105, H116 to H106, H103 to H107, H109 to H108, H117 to H109, H104 to H110, H110 to H111, H118 to H112, H105 to H113, H111 to H114, H119 to H115, H112 to H116, H120 to H117, H113 to H118, H121 to H119, H114 to H120, H122 to H121, H106 to H122, ICON102 to ICON101, ICON101 to ICON102
Changed lines of the file:
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@@
 (kicad_sch
-	(version 20231120)
+	(version 20250114)
 	(generator "eeschema")
-	(generator_version "8.0")
+	(generator_version "9.0")
 	(paper "A4")
 	(title_block
 		(title "V2 express")
-		(date "2023-01-09")
-		(rev "1")
+		(date "2025-10-27")
+		(rev "2")
 		(company "Versio Duo")
 		(comment 1 "cover")
@@
 		(dnp no)
 		(fields_autoplaced yes)
-		(property "Reference" "H118"
+		(property "Reference" "H112"
 			(at 190.5 64.7699 90)
 			(effects
@@
 			(project "express-cover"
 				(path "/6c8448b4-b04d-47e1-934e-e40cbe27a7be"
-					(reference "H118")
+					(reference "H112")
 					(unit 1)
 				)
@@
 		(dnp no)
 		(fields_autoplaced yes)
-		(property "Reference" "H110"
+		(property "Reference" "H111"
 			(at 140.97 64.7699 90)
 			(effects
@@
 			(project "express-cover"
 				(path "/6c8448b4-b04d-47e1-934e-e40cbe27a7be"
-					(reference "H110")
+					(reference "H111")
 					(unit 1)
 				)
@@
 		(dnp no)
 		(fields_autoplaced yes)
-		(property "Reference" "H109"
+		(property "Reference" "H108"
 			(at 140.97 57.1499 90)
 			(effects
@@
 			(project "express-cover"
 				(path "/6c8448b4-b04d-47e1-934e-e40cbe27a7be"
-					(reference "H109")
+					(reference "H108")
 					(unit 1)
 				)
@@
 		(dnp no)
 		(fields_autoplaced yes)
-		(property "Reference" "H103"
+		(property "Reference" "H107"
 			(at 88.9 57.785 90)
 			(effects
@@
 			(project "express-cover"
 				(path "/6c8448b4-b04d-47e1-934e-e40cbe27a7be"
-					(reference "H103")
+					(reference "H107")
 					(unit 1)
 				)
@@
 		(dnp no)
 		(fields_autoplaced yes)
-		(property "Reference" "H116"
+		(property "Reference" "H106"
 			(at 190.5 49.5299 90)
 			(effects
@@
 			(project "express-cover"
 				(path "/6c8448b4-b04d-47e1-934e-e40cbe27a7be"
-					(reference "H116")
+					(reference "H106")
 					(unit 1)
 				)
@@
 		(dnp no)
 		(fields_autoplaced yes)
-		(property "Reference" "H117"
+		(property "Reference" "H109"
 			(at 190.5 57.1499 90)
 			(effects
@@
 			(project "express-cover"
 				(path "/6c8448b4-b04d-47e1-934e-e40cbe27a7be"
-					(reference "H117")
+					(reference "H109")
 					(unit 1)
 				)
@@
 		(dnp no)
 		(fields_autoplaced yes)
-		(property "Reference" "H107"
+		(property "Reference" "H102"
 			(at 140.97 41.9099 90)
 			(effects
@@
 			(project "express-cover"
 				(path "/6c8448b4-b04d-47e1-934e-e40cbe27a7be"
-					(reference "H107")
+					(reference "H102")
 					(unit 1)
 				)
@@
 		(dnp no)
 		(fields_autoplaced yes)
-		(property "Reference" "H119"
+		(property "Reference" "H115"
 			(at 190.5 72.3899 90)
 			(effects
@@
 			(project "express-cover"
 				(path "/6c8448b4-b04d-47e1-934e-e40cbe27a7be"
-					(reference "H119")
+					(reference "H115")
 					(unit 1)
 				)
@@
 		(dnp no)
 		(fields_autoplaced yes)
-		(property "Reference" "H114"
+		(property "Reference" "H120"
 			(at 140.97 95.2499 90)
 			(effects
@@
 			(project "express-cover"
 				(path "/6c8448b4-b04d-47e1-934e-e40cbe27a7be"
-					(reference "H114")
+					(reference "H120")
 					(unit 1)
 				)
@@
 		(dnp no)
 		(fields_autoplaced yes)
-		(property "Reference" "H122"
+		(property "Reference" "H121"
 			(at 190.5 95.2499 90)
 			(effects
@@
 			(project "express-cover"
 				(path "/6c8448b4-b04d-47e1-934e-e40cbe27a7be"
-					(reference "H122")
+					(reference "H121")
 					(unit 1)
 				)
@@
 		(dnp no)
 		(fields_autoplaced yes)
-		(property "Reference" "H111"
+		(property "Reference" "H114"
 			(at 140.97 72.3899 90)
 			(effects
@@
 			(project "express-cover"
 				(path "/6c8448b4-b04d-47e1-934e-e40cbe27a7be"
-					(reference "H111")
+					(reference "H114")
 					(unit 1)
 				)
@@
 		(on_board yes)
 		(dnp no)
-		(property "Reference" "ICON101"
+		(property "Reference" "ICON102"
 			(at 105.41 146.05 0)
 			(effects
@@
 			(project "express-cover"
 				(path "/6c8448b4-b04d-47e1-934e-e40cbe27a7be"
-					(reference "ICON101")
+					(reference "ICON102")
 					(unit 1)
 				)
@@
 		(dnp no)
 		(fields_autoplaced yes)
-		(property "Reference" "H120"
+		(property "Reference" "H117"
 			(at 190.5 80.0099 90)
 			(effects
@@
 			(project "express-cover"
 				(path "/6c8448b4-b04d-47e1-934e-e40cbe27a7be"
-					(reference "H120")
+					(reference "H117")
 					(unit 1)
 				)
@@
 		(dnp no)
 		(fields_autoplaced yes)
-		(property "Reference" "H121"
+		(property "Reference" "H119"
 			(at 190.5 87.6299 90)
 			(effects
@@
 			(project "express-cover"
 				(path "/6c8448b4-b04d-47e1-934e-e40cbe27a7be"
-					(reference "H121")
+					(reference "H119")
 					(unit 1)
 				)
@@
 		(dnp no)
 		(fields_autoplaced yes)
-		(property "Reference" "H105"
+		(property "Reference" "H113"
 			(at 88.9 73.025 90)
 			(effects
@@
 			(project "express-cover"
 				(path "/6c8448b4-b04d-47e1-934e-e40cbe27a7be"
-					(reference "H105")
+					(reference "H113")
 					(unit 1)
 				)
@@
 		(dnp no)
 		(fields_autoplaced yes)
-		(property "Reference" "H102"
+		(property "Reference" "H104"
 			(at 88.9 50.165 90)
 			(effects
@@
 			(project "express-cover"
 				(path "/6c8448b4-b04d-47e1-934e-e40cbe27a7be"
-					(reference "H102")
+					(reference "H104")
 					(unit 1)
 				)
@@
 		(dnp no)
 		(fields_autoplaced yes)
-		(property "Reference" "H115"
+		(property "Reference" "H103"
 			(at 190.5 41.9099 90)
 			(effects
@@
 			(project "express-cover"
 				(path "/6c8448b4-b04d-47e1-934e-e40cbe27a7be"
-					(reference "H115")
+					(reference "H103")
 					(unit 1)
 				)
@@
 		(dnp no)
 		(fields_autoplaced yes)
-		(property "Reference" "H108"
+		(property "Reference" "H105"
 			(at 140.97 49.5299 90)
 			(effects
@@
 			(project "express-cover"
 				(path "/6c8448b4-b04d-47e1-934e-e40cbe27a7be"
-					(reference "H108")
+					(reference "H105")
 					(unit 1)
 				)
@@
 		(dnp no)
 		(fields_autoplaced yes)
-		(property "Reference" "H112"
+		(property "Reference" "H116"
 			(at 140.97 80.0099 90)
 			(effects
@@
 			(project "express-cover"
 				(path "/6c8448b4-b04d-47e1-934e-e40cbe27a7be"
-					(reference "H112")
+					(reference "H116")
 					(unit 1)
 				)
@@
 		(dnp no)
 		(fields_autoplaced yes)
-		(property "Reference" "H113"
+		(property "Reference" "H118"
 			(at 140.97 87.6299 90)
 			(effects
@@
 			(project "express-cover"
 				(path "/6c8448b4-b04d-47e1-934e-e40cbe27a7be"
-					(reference "H113")
+					(reference "H118")
 					(unit 1)
 				)
@@
 		(dnp no)
 		(fields_autoplaced yes)
-		(property "Reference" "H106"
+		(property "Reference" "H122"
 			(at 88.9 121.9199 0)
 			(effects
@@
 			(project "express-cover"
 				(path "/6c8448b4-b04d-47e1-934e-e40cbe27a7be"
-					(reference "H106")
+					(reference "H122")
 					(unit 1)
 				)
@@
 		(on_board yes)
 		(dnp no)
-		(property "Reference" "ICON102"
+		(property "Reference" "ICON101"
 			(at 83.185 144.78 0)
 			(effects
@@
 			(project "express-cover"
 				(path "/6c8448b4-b04d-47e1-934e-e40cbe27a7be"
-					(reference "ICON102")
+					(reference "ICON101")
 					(unit 1)
 				)
@@
 		(dnp no)
 		(fields_autoplaced yes)
-		(property "Reference" "H104"
+		(property "Reference" "H110"
 			(at 88.9 65.405 90)
 			(effects
@@
 			(project "express-cover"
 				(path "/6c8448b4-b04d-47e1-934e-e40cbe27a7be"
-					(reference "H104")
+					(reference "H110")
 					(unit 1)
 				)
@@
 		)
 	)
+	(embedded_fonts no)
 )
